Commit message: updated keyboard control code and urdf

File: urdf/truck_urdf.urdf.xacro (robot description, xacro)
@@ -66,5 +66,5 @@
       <surface>
         <contact><ode><kp>1e6</kp><kd>1.0</kd><max_vel>0.2</max_vel><min_depth>0.001</min_depth></ode></contact>
-        <friction><ode><mu>3.2</mu><mu2>3.2</mu2><slip1>0.01</slip1><slip2>0.0</slip2></ode></friction>
+        <friction><ode><mu>2.0</mu><mu2>2.0</mu2><slip1>0.05</slip1><slip2>0.05</slip2></ode></friction>
       </surface>
     </collision>
@@ -108,5 +108,5 @@
       <surface>
         <contact><ode><kp>1e6</kp><kd>1.0</kd><max_vel>0.2</max_vel><min_depth>0.001</min_depth></ode></contact>
-        <friction><ode><mu>3.2</mu><mu2>3.2</mu2><slip1>0.01</slip1><slip2>0.0</slip2></ode></friction>
+        <friction><ode><mu>2.0</mu><mu2>2.0</mu2><slip1>0.05</slip1><slip2>0.05</slip2></ode></friction>
       </surface>
     </collision>
@@ -133,5 +133,5 @@
       <surface>
         <contact><ode><kp>1e6</kp><kd>1.0</kd><max_vel>0.2</max_vel><min_depth>0.001</min_depth></ode></contact>
-        <friction><ode><mu>7.2</mu><mu2>7.2</mu2><slip1>0.01</slip1><slip2>0.0</slip2></ode></friction>
+        <friction><ode><mu>3.0</mu><mu2>3.0</mu2><slip1>0.02</slip1><slip2>0.02</slip2></ode></friction>
       </surface>
     </collision>
@@ -157,5 +157,5 @@
       <surface>
         <contact><ode><kp>1e6</kp><kd>1.0</kd><max_vel>0.2</max_vel><min_depth>0.001</min_depth></ode></contact>
-        <friction><ode><mu>7.2</mu><mu2>7.2</mu2><slip1>0.01</slip1><slip2>0.0</slip2></ode></friction>
+        <friction><ode><mu>3.0</mu><mu2>3.0</mu2><slip1>0.02</slip1><slip2>0.02</slip2></ode></friction>
       </surface>
     </collision>
@@ -184,5 +184,5 @@
   <!-- keep your original pose -->
   <origin xyz="-0.254000000000682 -1.06680000000062 -0.20320000000001"
-          rpy="-3.14159265358979 0 -0.0250798506762473"/>
+          rpy="-3.14159265358979 0 0"/>
   <parent link="base_link"/>
   <child  link="trailer"/>
@@ -190,7 +190,7 @@
   <axis xyz="0 0 1"/>
   <!-- turn limits (tweak as you like) -->
-  <limit lower="-1.2" upper="1.2" effort="500.0" velocity="2.0"/>
+  <limit lower="-1.5" upper="1.5" effort="500.0" velocity="3.0"/>
   <!-- add some damping so it’s stable -->
-  <dynamics damping="5.0" friction="0.0"/>
+  <dynamics damping="1.0" friction="0.0"/>
   </joint>
   <!-- Trailer wheels: all free-rolling (continuous, axle along X) -->
@@ -204,6 +204,6 @@
       <geometry><cylinder radius="0.17" length="0.06"/></geometry>
       <surface>
-        <contact><ode><kp>1e6</kp><kd>1.0</kd><max_vel>0.2</max_vel><min_depth>0.001</min_depth></ode></contact>
-        <friction><ode><mu>1.0</mu><mu2>1.0</mu2><slip1>0.01</slip1><slip2>0.0</slip2></ode></friction>
+        <contact><ode><kp>5e5</kp><kd>5.0</kd><max_vel>0.5</max_vel><min_depth>0.001</min_depth></ode></contact>
+        <friction><ode><mu>0.8</mu><mu2>0.3</mu2><slip1>0.1</slip1><slip2>0.1</slip2></ode></friction>
       </surface>
     </collision>
@@ -223,6 +223,6 @@
       <geometry><cylinder radius="0.17" length="0.06"/></geometry>
       <surface>
-        <contact><ode><kp>1e6</kp><kd>1.0</kd><max_vel>0.2</max_vel><min_depth>0.001</min_depth></ode></contact>
-        <friction><ode><mu>1.0</mu><mu2>1.0</mu2><slip1>0.01</slip1><slip2>0.0</slip2></ode></friction>
+        <contact><ode><kp>5e5</kp><kd>5.0</kd><max_vel>0.5</max_vel><min_depth>0.001</min_depth></ode></contact>
+        <friction><ode><mu>0.8</mu><mu2>0.3</mu2><slip1>0.1</slip1><slip2>0.1</slip2></ode></friction>
       </surface>
     </collision>
@@ -242,6 +242,6 @@
       <geometry><cylinder radius="0.17" length="0.06"/></geometry>
       <surface>
-        <contact><ode><kp>1e6</kp><kd>1.0</kd><max_vel>0.2</max_vel><min_depth>0.001</min_depth></ode></contact>
-        <friction><ode><mu>1.0</mu><mu2>1.0</mu2><slip1>0.01</slip1><slip2>0.0</slip2></ode></friction>
+        <contact><ode><kp>5e5</kp><kd>5.0</kd><max_vel>0.5</max_vel><min_depth>0.001</min_depth></ode></contact>
+        <friction><ode><mu>0.8</mu><mu2>0.3</mu2><slip1>0.1</slip1><slip2>0.1</slip2></ode></friction>
       </surface>
     </collision>
@@ -261,6 +261,6 @@
       <geometry><cylinder radius="0.17" length="0.06"/></geometry>
       <surface>
-        <contact><ode><kp>1e6</kp><kd>1.0</kd><max_vel>0.2</max_vel><min_depth>0.001</min_depth></ode></contact>
-        <friction><ode><mu>1.0</mu><mu2>1.0</mu2><slip1>0.01</slip1><slip2>0.0</slip2></ode></friction>
+        <contact><ode><kp>5e5</kp><kd>5.0</kd><max_vel>0.5</max_vel><min_depth>0.001</min_depth></ode></contact>
+        <friction><ode><mu>0.8</mu><mu2>0.3</mu2><slip1>0.1</slip1><slip2>0.1</slip2></ode></friction>
       </surface>
     </collision>
@@ -285,10 +285,10 @@
   </link>
   <joint name="back_hitch" type="revolute">
-  <origin xyz="0 1.15526871138527 0" rpy="0 0 -0.0257409734881418"/>
+  <origin xyz="0 1.15526871138527 0" rpy="0 0 0"/>
   <parent link="trailer"/>
   <child  link="back_trailer"/>
   <axis xyz="0 0 1"/>
-  <limit lower="-1.2" upper="1.2" effort="500.0" velocity="2.0"/>
-  <dynamics damping="5.0" friction="0.0"/>
+  <limit lower="-1.5" upper="1.5" effort="500.0" velocity="3.0"/>
+  <dynamics damping="1.0" friction="0.0"/>
   </joint>
   <!-- Back trailer wheels: free-rolling -->
@@ -302,6 +302,6 @@
       <geometry><cylinder radius="0.17" length="0.06"/></geometry>
       <surface>
-        <contact><ode><kp>1e6</kp><kd>1.0</kd><max_vel>0.2</max_vel><min_depth>0.001</min_depth></ode></contact>
-        <friction><ode><mu>1.0</mu><mu2>1.0</mu2><slip1>0.01</slip1><slip2>0.0</slip2></ode></friction>
+        <contact><ode><kp>5e5</kp><kd>5.0</kd><max_vel>0.5</max_vel><min_depth>0.001</min_depth></ode></contact>
+        <friction><ode><mu>0.8</mu><mu2>0.3</mu2><slip1>0.1</slip1><slip2>0.1</slip2></ode></friction>
       </surface>
     </collision>
@@ -321,6 +321,6 @@
       <geometry><cylinder radius="0.17" length="0.06"/></geometry>
       <surface>
-        <contact><ode><kp>1e6</kp><kd>1.0</kd><max_vel>0.2</max_vel><min_depth>0.001</min_depth></ode></contact>
-        <friction><ode><mu>1.0</mu><mu2>1.0</mu2><slip1>0.01</slip1><slip2>0.0</slip2></ode></friction>
+        <contact><ode><kp>5e5</kp><kd>5.0</kd><max_vel>0.5</max_vel><min_depth>0.001</min_depth></ode></contact>
+        <friction><ode><mu>0.8</mu><mu2>0.3</mu2><slip1>0.1</slip1><slip2>0.1</slip2></ode></friction>
       </surface>
     </collision>
@@ -340,6 +340,6 @@
       <geometry><cylinder radius="0.17" length="0.06"/></geometry>
       <surface>
-        <contact><ode><kp>1e6</kp><kd>1.0</kd><max_vel>0.2</max_vel><min_depth>0.001</min_depth></ode></contact>
-        <friction><ode><mu>1.0</mu><mu2>1.0</mu2><slip1>0.01</slip1><slip2>0.0</slip2></ode></friction>
+        <contact><ode><kp>5e5</kp><kd>5.0</kd><max_vel>0.5</max_vel><min_depth>0.001</min_depth></ode></contact>
+        <friction><ode><mu>0.8</mu><mu2>0.3</mu2><slip1>0.1</slip1><slip2>0.1</slip2></ode></friction>
       </surface>
     </collision>
@@ -359,6 +359,6 @@
       <geometry><cylinder radius="0.17" length="0.06"/></geometry>
       <surface>
-        <contact><ode><kp>1e6</kp><kd>1.0</kd><max_vel>0.2</max_vel><min_depth>0.001</min_depth></ode></contact>
-        <friction><ode><mu>1.0</mu><mu2>1.0</mu2><slip1>0.01</slip1><slip2>0.0</slip2></ode></friction>
+        <contact><ode><kp>5e5</kp><kd>5.0</kd><max_vel>0.5</max_vel><min_depth>0.001</min_depth></ode></contact>
+        <friction><ode><mu>0.8</mu><mu2>0.3</mu2><slip1>0.1</slip1><slip2>0.1</slip2></ode></friction>
       </surface>
     </collision>

Commit message: lidar tweaks

File: urdf/truck_urdf.urdf.xacro (robot description, xacro)
@@ -382,5 +382,5 @@
       <cylinder radius="0.03" length="0.06"/>
     </geometry>
-    <material><color rgba="0.1 0.1 0.1 1.0"/></material>
+    <material name="lidar_mat"><color rgba="0.1 0.1 0.1 1.0"/></material>
   </visual>
 </link>
@@ -388,5 +388,5 @@
 <joint name="lidar_mount" type="fixed">
   <!-- Shift slightly forward and upward -->
-  <origin xyz="0.25 0.0 0.45" rpy="0 0 0"/>
+  <origin xyz="0 0.0 0.8" rpy="0 0 0"/>
   <parent link="base_link"/>
   <child link="lidar_link"/>
@@ -396,5 +396,5 @@
   <sensor name="lidar" type="ray">
     <!-- Adjusted pose -->
-    <pose>0 0 0.03 0 1.5708 0</pose>
+    <pose>0 0 0 0 0 0</pose>
     <always_on>true</always_on>
     <visualize>true</visualize>
